File: board_a/board_a.kicad_pcb (KiCad board)
At the start: 2 copper layers, 29.3 x 26.2 mm, 15 parts, among them J1 Shuttle 3.0 sockets, J2 2x8 header, J3 IDD meter

Commit message: Boards A and B: drop the JLCJLCJLCJLC order-number placeholder
JLCPCB now removes its order mark for free by default ("Mark on PCB:
Remove Mark"), so the placeholder would have been printed as text.
Gerbers regenerated; DRC still 0.

Co-Authored-By: Claude Opus 5.5 <noreply@anthropic.com>
Other:
- board text removed: "JLCJLCJLCJLC"
