File: board_b/board_b.kicad_pcb (KiCad board)
At the start: 2 copper layers, 25.5 x 24.6 mm, 16 parts, among them J1 Shuttle 3.0 sockets, J3 IDD meter, U1 XIAO ESP32S3

Commit message: Boards A and B: drop the JLCJLCJLCJLC order-number placeholder
JLCPCB now removes its order mark for free by default ("Mark on PCB:
Remove Mark"), so the placeholder would have been printed as text.
Gerbers regenerated; DRC still 0.

Co-Authored-By: Claude Opus 5.5 <noreply@anthropic.com>
Other:
- board text removed: "JLCJLCJLCJLC"
